Commit message: controller loaded

File: urdf/zumy.xacro (robot description, xacro)
@@ -15,5 +15,5 @@
   <xacro:property name="wheel_pos_x" value="0.15"/>
   <xacro:property name="caster_radius" value="0.1"/>
-  <!--xacro:include filename="$(find zumy_description)/urdf/zumy.gazebo" /-->
+  <xacro:include filename="$(find zumy_description)/urdf/zumy.gazebo" />
   <link name="base_link">
     <visual>
@@ -139,3 +139,24 @@
     <origin xyz="0.105 0 0.22" rpy="0 0 0"/>
   </joint-->
+  <!-- URDF and ros control bridge-->
+  <transmission name="tran1">
+    <type>transmission_interface/SimpleTransmission</type>
+    <joint name="base_to_lwheel">
+      <hardwareInterface>EffortJointInterface</hardwareInterface>
+    </joint>
+    <actuator name="motor1">
+      <!--hardwareInterface>EffortJointInterface</hardwareInterface-->
+      <mechanicalReduction>1</mechanicalReduction>
+    </actuator>
+  </transmission>
+  <transmission name="tran2">
+    <type>transmission_interface/SimpleTransmission</type>
+    <joint name="base_to_rwheel">
+      <hardwareInterface>EffortJointInterface</hardwareInterface>
+    </joint>
+    <actuator name="motor2">
+      <!--hardwareInterface>EffortJointInterface</hardwareInterface-->
+      <mechanicalReduction>1</mechanicalReduction>
+    </actuator>
+  </transmission>
 </robot>

Commit message: collision origin fixed

File: urdf/zumy.xacro (robot description, xacro)
@@ -8,10 +8,8 @@
   <xacro:property name="chasis_height" value="0.1"/>
   <xacro:property name="wheel_thickness" value="0.03"/>
-  <xacro:property name="wheel_radius" value="0.15"/>
-  <!--value = ${chasis_height}-->
-  <xacro:property name="wheel_center_height" value="0.1"/>
-  <!--value = $(body_width + wheel_thickness/2)/2+0.05-->
-  <xacro:property name="wheel_center_y" value="0.7"/>
-  <xacro:property name="wheel_pos_x" value="0.15"/>
+  <xacro:property name="wheel_radius" value="0.1"/>
+  <xacro:property name="wheel_center_height" value="${chasis_height}"/>
+  <xacro:property name="wheel_center_y" value="${(body_width+wheel_thickness)/2}"/>
+  <xacro:property name="wheel_center_x" value="0.1"/>
   <xacro:property name="caster_radius" value="0.1"/>
   <xacro:include filename="$(find zumy_description)/urdf/zumy.gazebo" />
@@ -39,4 +37,5 @@
         <box size="${body_length} ${body_width} ${body_height}"/>
       </geometry>
+      <origin rpy="0 0 0" xyz="0 0 ${chasis_height}"/>
     </collision>
   <collision name='caster_collision'>
@@ -78,4 +77,5 @@
         <cylinder length="${wheel_thickness}" radius="${wheel_radius}"/>
       </geometry>
+      <origin rpy="0 1.5707 1.5707" xyz="0 ${-wheel_center_y} 0"/>
     </collision>
     <inertial>
@@ -90,5 +90,5 @@
     <parent link="base_link"/>
     <child link="lwheel"/>
-    <origin xyz="${wheel_pos_x} 0 ${wheel_center_height}" rpy="0 0 0"/>
+    <origin xyz="${wheel_center_x} 0 ${wheel_center_height}" rpy="0 0 0"/>
     <axis xyz="0 1 0"/>
   </joint>
@@ -107,7 +107,8 @@
         <cylinder length="${wheel_thickness}" radius="${wheel_radius}"/>
       </geometry>
+      <origin rpy="0 1.5707 1.5707" xyz="0 ${wheel_center_y} 0"/>
     </collision>
     <inertial>
-      <origin xyz="0 0 1" rpy="0 0 0"/>
+      <!--origin xyz="0 0 1" rpy="0 0 0"/-->
       <mass value="1"/>
       <inertia
@@ -120,5 +121,5 @@
     <parent link="base_link"/>
     <child link="rwheel"/>
-    <origin xyz="${wheel_pos_x} 0 ${wheel_center_height}" rpy="0 0 0"/>
+    <origin xyz="${wheel_center_x} 0 ${wheel_center_height}" rpy="0 0 0"/>
     <axis xyz="0 1 0"/>
   </joint>

Commit message: better caster urdf

File: urdf/zumy.xacro (robot description, xacro)
@@ -56,5 +56,5 @@
   </collision>
     <inertial>
-      <mass value="1"/>
+      <mass value="50"/>
       <inertia
 	  ixx="1.0" ixy="0.0" ixz="0.0"
